Commit message: Add camera-mounted gripper body + D435 URDF integration
- usd/parts/gripper_body_camera.stl: new gripper body with D435 camera housing
- usd/parts/gripper_body_camera_urdf.stl: URDF-coordinate version (Y-offset applied)
- gripper_assembly.urdf: replaced mesh → gripper_body_camera_urdf.stl,
  added camera_joint (xyz="-0.0402 -0.0855 -0.0676" rpy="2.3562 0 0")
  and camera_color_optical_frame link
- gripper_body.urdf: mesh updated to gripper_body_camera_urdf.stl
- camera_view.py, capture.py: RealSense D435 viewer/capture tools
- cube_analysis.py: HSV cube detection + edge sharpness pipeline
- output/front|side|top.png: gripper CAD reference views
- output/gripper_3view_v8.png: final 3-view assembly diagram
  (lens: X=5, Y=-95, Z=-42mm, dir: -Y+Z 45°)

Co-Authored-By: Claude Sonnet 4.6 <noreply@anthropic.com>

File: usd/parts/gripper_assembly.urdf (robot description, URDF)
Before this commit: robot gripper_assembly, 3 links, 2 joints
Links:
- added link camera_color_optical_frame
- added link camera_link
- link gripper_base_link: geometry collision mesh filename=gripper_body_camera_urdf.stl scale=0.001 0.001 0.001; visual mesh filename=gripper_body_camera_urdf.stl scale=0.001 0.001 0.001
Joints:
- added joint camera_color_optical_joint: type fixed, parent camera_link, child camera_color_optical_frame, origin xyz=0 0 0 rpy=-1.5708 0 -1.5708
- added joint camera_joint: type fixed, parent gripper_base_link, child camera_link, origin xyz=-0.0402 -0.0855 -0.0676 rpy=2.3562 0 0

File: usd/parts/gripper_body.urdf (robot description, URDF)
Before this commit: robot gripper_body, 1 links, 0 joints
Links:
- link gripper_body_link: geometry collision mesh filename=gripper_body_camera_urdf.stl scale=0.001 0.001 0.001; visual mesh filename=gripper_body_camera_urdf.stl scale=0.001 0.001 0.001
